File: DE10-Nano/ST-DC1 daughtercard/HW/kicad/file5D22A4F0.sch (KiCad schematic (older format))
At the start: 8 parts, among them J46 Conn_RS422, U19 74LVC2G04, U3 DS89C21

Commit message: Add Artwork to PCB:   DE10-Nano/ST-DC1 daughtercard/HW/kicad/DE10nano interface-cache.lib 	Add Artwork to PCB:    DE10-Nano/ST-DC1 daughtercard/HW/kicad/DE10nano interface.jpg 	Add termination Resistors to diff inputs:   DE10-Nano/ST-DC1 daughtercard/HW/kicad/DE10nano interface.kicad_pcb 	Add termination Resistors to diff inputs:   DE10-Nano/ST-DC1 daughtercard/HW/kicad/DE10nano interface.kicad_pcb-bak 	Add termination Resistors to diff inputs:   DE10-Nano/ST-DC1 daughtercard/HW/kicad/DE10nano interface.net 	Add termination Resistors to diff inputs:   DE10-Nano/ST-DC1 daughtercard/HW/kicad/DE10nano interface.pro 	Add termination Resistors to diff inputs:   DE10-Nano/ST-DC1 daughtercard/HW/kicad/Images/DE10nano interface back.jpg 	Add Artwork to PCB:   DE10-Nano/ST-DC1 daughtercard/HW/kicad/Images/DE10nano interface.jpg 	Reflect incomplete BOM:    DE10-Nano/ST-DC1 daughtercard/HW/kicad/bom/BOM.ods -> DE10-Nano/ST-DC1 daughtercard/HW/kicad/bom/BOM-incomplete-use-ibom.ods 	Add termination Resistors to diff inputs:   DE10-Nano/ST-DC1 daughtercard/HW/kicad/bom/ibom.html 	Add termination Resistors to diff inputs:   DE10-Nano/ST-DC1 daughtercard/HW/kicad/file5CE4621E.sch 	Add termination Resistors to diff inputs:   DE10-Nano/ST-DC1 daughtercard/HW/kicad/file5CE4621E.sch-bak 	Add termination Resistors to diff inputs:   DE10-Nano/ST-DC1 daughtercard/HW/kicad/file5D10B445.sch-bak 	Add termination Resistors to diff inputs:   DE10-Nano/ST-DC1 daughtercard/HW/kicad/file5D22A4F0.sch 	modified:   DE10-Nano/ST-DC1 daughtercard/HW/kicad/file5D22A4F0.sch-bak 	modified:   DE10-Nano/ST-DC1 daughtercard/HW/kicad/gerbers rev_G.zip 	modified:   DE10-Nano/ST-DC1 daughtercard/HW/kicad/gerbers rev_G/DE10nano interface-B_Cu.gbr 	modified:   DE10-Nano/ST-DC1 daughtercard/HW/kicad/gerbers rev_G/DE10nano interface-B_Mask.gbr 	modified:   DE10-Nano/ST-DC1 daughtercard/HW/kicad/gerbers rev_G/DE10nano interface-B_Paste.gbr 	modified:   DE10-Nano/ST-DC1 daughtercard/HW/kicad/gerbers rev_G/DE10nano i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
Parts:
- removed R2: 120R, Resistor_SMD:R_0805_2012Metric_Pad1.15x1.40mm_HandSolder, symbol DE10nano-interface-rescue:R_Small-Device
Changed lines of the file:
@@
 	4700 2700 4700 3150
-$Comp
-L DE10nano-interface-rescue:R_Small-Device R7
-U 1 1 5D22AC57
-P 5800 3300
-F 0 "R7" H 5600 3350 50  0000 L CNN
-F 1 "120R" H 5550 3250 50  0000 L CNN
-F 2 "Resistor_SMD:R_0805_2012Metric_Pad1.15x1.40mm_HandSolder" H 5800 3300 50  0001 C CNN
-F 3 "~" H 5800 3300 50  0001 C CNN
-	1    5800 3300
-	1    0    0    -1
-$EndComp
 $Comp
 L DE10nano-interface-rescue:C_Small-Device C9
@@
 $EndComp
 Wire Wire Line
-	5800 3200 5800 2950
-Wire Wire Line
-	5800 2950 6300 2950
-Wire Wire Line
-	5800 3400 5800 3650
-Wire Wire Line
-	5800 3650 6300 3650
-Wire Wire Line
 	6050 3300 6150 3300
 Wire Wire Line
@@
 Connection ~ 6050 4200
 Wire Wire Line
-	5800 3650 5100 3650
-Connection ~ 5800 3650
-Wire Wire Line
-	5800 2950 5350 2950
-Wire Wire Line
 	5350 2950 5350 3450
 Wire Wire Line
 	5350 3450 5100 3450
-Connection ~ 5800 2950
 Wire Wire Line
 	5100 4050 5350 4050
@@
 Wire Wire Line
 	3900 2350 4700 2350
-Wire Wire Line
-	5350 4550 5800 4550
-Wire Wire Line
-	5800 4550 6300 4550
-Connection ~ 5800 4550
-Wire Wire Line
-	5800 4300 5800 4550
-Wire Wire Line
-	5800 3850 5100 3850
-Wire Wire Line
-	5800 3850 6300 3850
-Connection ~ 5800 3850
-Wire Wire Line
-	5800 4100 5800 3850
-$Comp
-L DE10nano-interface-rescue:R_Small-Device R2
-U 1 1 5D2C9361
-P 5800 4200
-F 0 "R2" H 5900 4150 50  0000 L CNN
-F 1 "120R" H 5850 4250 50  0000 L CNN
-F 2 "Resistor_SMD:R_0805_2012Metric_Pad1.15x1.40mm_HandSolder" H 5800 4200 50  0001 C CNN
-F 3 "~" H 5800 4200 50  0001 C CNN
-	1    5800 4200
-	-1   0    0    1
-$EndComp
 Text Label 7600 4000 2    50   ~ 0
 GND
@@
 	1    0    0    -1
 $EndComp
+Wire Wire Line
+	5800 3650 5100 3650
+Wire Wire Line
+	5800 3650 6300 3650
+Connection ~ 5800 3650
+Wire Wire Line
+	5800 3400 5800 3650
+Wire Wire Line
+	5800 2950 5350 2950
+Wire Wire Line
+	5800 2950 6300 2950
+Connection ~ 5800 2950
+Wire Wire Line
+	5800 3200 5800 2950
+$Comp
+L DE10nano-interface-rescue:R_Small-Device R7
+U 1 1 5D22AC57
+P 5800 3300
+F 0 "R7" H 5600 3350 50  0000 L CNN
+F 1 "120R" H 5550 3250 50  0000 L CNN
+F 2 "Resistor_SMD:R_0805_2012Metric_Pad1.15x1.40mm_HandSolder" H 5800 3300 50  0001 C CNN
+F 3 "~" H 5800 3300 50  0001 C CNN
+	1    5800 3300
+	1    0    0    -1
+$EndComp
+Wire Wire Line
+	5350 4550 6300 4550
+Wire Wire Line
+	5100 3850 6300 3850
 $EndSCHEMATC
